File: hardware/squall-led-shield/squall-led-shield.sch (KiCad schematic (older format))
At the start: 10 parts, among them J1 SQUALL_HEADER, Q1 Q_2NMOS

Commit message: Add missing footprint for R2
Parts:
- R2: footprint (none) -> Resistors_SMD:R_0603
Changed lines of the file:
@@
 F 0 "R2" V 2757 5000 50  0000 C CNN
 F 1 "18Ω" V 2666 5000 50  0000 C CNN
-F 2 "" V 2480 5000 50  0000 C CNN
+F 2 "Resistors_SMD:R_0603" V 2480 5000 50  0001 C CNN
 F 3 "" H 2550 5000 50  0000 C CNN
 	1    2550 5000
